File: Pi_relay1.sch (KiCad schematic (older format))
At the start: 7 parts, among them K1 G5Q-1, Q1 2N7002

Commit message: Button added
Parts:
- D1: footprint Diode_SMD:D_SOD-123 -> Diode_SMD:D_SOD-323
- R1: value 2K -> 1K
- R3: renamed from R4; value 100 -> 200
- renumbered D3 to D2
Changed lines of the file:
@@
 $Descr A4 11693 8268
 encoding utf-8
-Sheet 2 3
+Sheet 2 2
 Title ""
 Date ""
@@
 F 0 "D1" H 5050 4750 50  0000 C CNN
 F 1 "B5818WS" H 5050 4550 50  0000 C CNN
-F 2 "Diode_SMD:D_SOD-123" H 5050 4650 50  0001 C CNN
+F 2 "Diode_SMD:D_SOD-323" H 5050 4650 50  0001 C CNN
 F 3 "" H 5050 4650 50  0001 C CNN
 	1    5050 4650
@@
 P 4200 5500
 F 0 "R1" V 3993 5500 50  0000 C CNN
-F 1 "2K" V 4084 5500 50  0000 C CNN
+F 1 "1K" V 4084 5500 50  0000 C CNN
 F 2 "Resistor_SMD:R_0805_2012Metric" V 4130 5500 50  0001 C CNN
 F 3 "~" H 4200 5500 50  0001 C CNN
@@
 AC_RELAY1
 $Comp
-L Device:R R4
+L Device:R R3
 U 1 1 5CEF18DD
 P 5150 5000
-F 0 "R4" V 5250 5000 50  0000 C CNN
-F 1 "100" V 5150 5000 50  0000 C CNN
+F 0 "R3" V 5250 5000 50  0000 C CNN
+F 1 "200" V 5150 5000 50  0000 C CNN
 F 2 "Resistor_SMD:R_0805_2012Metric" V 5080 5000 50  0001 C CNN
 F 3 "~" H 5150 5000 50  0001 C CNN
@@
 	5300 5000 5300 5300
 $Comp
-L Device:LED D3
+L Device:LED D2
 U 1 1 5CEF1975
 P 4850 5000
-F 0 "D3" H 4850 5100 50  0000 C CNN
+F 0 "D2" H 4850 5100 50  0000 C CNN
 F 1 "2.4/25" H 4850 4900 50  0000 C CNN
 F 2 "LED_SMD:LED_1206_3216Metric" H 4850 5000 50  0001 C CNN
