File: RPi_relays.sch (KiCad schematic (older format))
At the start: 7 parts, among them J1 Raspberry_Pi_2_3, J2 Conn_02x09_Odd_Even, J3 Conn_01x03_Female, J4 Conn_01x03_Female, J5 Conn_01x03_Female

Commit message: Button added
Parts:
- removed J2: Conn_02x09_Odd_Even, Connector_PinSocket_2.54mm:PinSocket_2x09_P2.54mm_Vertical, symbol Connector_Generic:Conn_02x09_Odd_Even
- removed J3, J4: Conn_01x03_Female, TerminalBlock:TerminalBlock_bornier-3_P5.08mm, symbol Connector:Conn_01x03_Female
- removed R3: 10K, Resistor_SMD:R_0805_2012Metric, symbol Device:R
- added F2: 50mA, Littelfuse:Littelfuse_LVR008NS, symbol Device:Polyfuse
- added J2: Conn_01x04_Female, Connector_Molex:Molex_Micro-Fit_3.0_43045-0412_2x02_P3.00mm_Vertical, symbol Connector:Conn_01x04_Female
- added U1: HLK-PMxx, Hi-Link:HLK-PM01, symbol hi-link:HLK-PMxx
- J1: renamed from J5; value Conn_01x03_Female -> PWR; footprint LP_connectors:PX0580_PC -> TerminalBlock_MetzConnect:TerminalBlock_MetzConnect_Type094_RT03504HBLU_1x04_P5.00mm_Horizontal; symbol Connector:Conn_01x03_Female -> Connector:Conn_01x04_Female
- renumbered J1 to J3
Connections:
- net 3V3: now also J2.2 (Pin_2); no longer J3.1 (3V3)
- net 5V: now also U1.3 (DC+)
- net AC_H: now also F1.1; no longer F1.2
- net AC_RELAY1: now also J1.1 (Pin_1)
- net GND: now also J1.3 (Pin_3), J2.1 (Pin_1), U1.4 (DC-)
- net RELAY1: now also J3.37 (GPIO26); no longer J3.16 (GPIO23)
- net DTRT_SW: now reaches J3.35 (GPIO19/MISO1)
- net DTRT_SW: now also J2.3 (Pin_3)
- net at J1.2 (Pin_2): now also U1.1 (AC_H)
- net D0: no longer names the net of J3.26 (~CE1~/GPIO7)
- net D1: no longer names the net of J3.24 (~CE0~/GPIO8)
- net D2: no longer names the net of J3.21 (MISO0/GPIO9)
- net D3: no longer names the net of J3.19 (MOSI0/GPIO10)
- net D4: no longer names the net of J3.23 (SCLK0/GPIO11)
- net D5: no longer names the net of J3.32 (PWM0/GPIO12)
- net D6 renamed DTRT_LED
- net DTRT_LED: now also J2.4 (Pin_4)
- net D7: no longer names the net of J3.8 (GPIO14/TXD)
- net HREF: no longer names the net of J3.7 (GCLK0/GPIO4)
- net PCLK: no longer names the net of J3.31 (GCLK2/GPIO6)
- net PWDN: no longer names the net of J3.36 (GPIO16)
- net RELAY2: no longer names the net of J3.22 (GPIO25)
- net RESET: no longer names the net of J3.10 (GPIO15/RXD)
- net SCL: no longer names the net of J3.5 (SCL/GPIO3)
- net SDA: no longer names the net of J3.3 (SDA/GPIO2)
- net VSYNC: no longer names the net of J3.29 (GCLK1/GPIO5)
- new net: F1.2, F2.2, J1.4 (Pin_4)
- new net: F2.1, U1.2 (AC_N)
- no-connect marks 1 -> 0
Other:
- moved on the sheet: F1
